Commit message: Add: env variables (fps, width, height)

File: src/ur10e_scene/urdf/realsense_d435.xacro (robot description, xacro)
@@ -1,4 +1,7 @@
 <?xml version="1.0"?>
 <robot xmlns:xacro="http://ros.org/wiki/xacro">
+  <xacro:property name="cam_fps" value="$(env TARGET_VIDEO_FPS)" />
+  <xacro:property name="cam_width" value="$(env TARGET_VIDEO_WIDTH)" />
+  <xacro:property name="cam_height" value="$(env TARGET_VIDEO_HEIGHT)" />
   <xacro:macro name="realsense_d435" params="parent *origin">
     <link name="camera_link">
@@ -37,10 +40,10 @@
       <sensor type="depth" name="camera">
         <always_on>true</always_on>
-        <update_rate>30.0</update_rate>
+        <update_rate>${cam_fps}</update_rate>
         <camera>
           <horizontal_fov>1.50098</horizontal_fov> <!-- Около 86 градусов (как у D435) -->
           <image>
-            <width>640</width>
-            <height>480</height>
+            <width>${cam_width}</width>
+            <height>${cam_height}</height>
             <format>B8G8R8</format>
           </image>

Commit message: Add: add YOLO-World perception pipeline

File: src/ur10e_scene/urdf/realsense_d435.xacro (robot description, xacro)
@@ -4,6 +4,6 @@
   <xacro:property name="cam_width" value="$(optenv TARGET_VIDEO_WIDTH 640)" />
   <xacro:property name="cam_height" value="$(optenv TARGET_VIDEO_HEIGHT 480)" />
-  <xacro:macro name="realsense_d435" params="parent *origin">
-    <link name="camera_link">
+  <xacro:macro name="realsense_d435" params="parent prefix:='camera' ros_namespace:='camera' camera_name:='camera' *origin">
+    <link name="${prefix}_link">
       <visual>
         <origin xyz="0 0 0" rpy="0 0 0"/>
@@ -26,17 +26,17 @@
       </inertial>
     </link>
-    <joint name="camera_joint" type="fixed">
+    <joint name="${prefix}_joint" type="fixed">
       <xacro:insert_block name="origin" />
       <parent link="${parent}"/>
-      <child link="camera_link"/>
+      <child link="${prefix}_link"/>
     </joint>
-    <link name="camera_color_optical_frame"/>
-    <joint name="camera_optical_joint" type="fixed">
+    <link name="${prefix}_color_optical_frame"/>
+    <joint name="${prefix}_optical_joint" type="fixed">
       <origin xyz="0 0 0" rpy="-1.57079632679 0 -1.57079632679"/>
-      <parent link="camera_link"/>
-      <child link="camera_color_optical_frame"/>
+      <parent link="${prefix}_link"/>
+      <child link="${prefix}_color_optical_frame"/>
     </joint>
-    <gazebo reference="camera_link">
-      <sensor type="depth" name="camera">
+    <gazebo reference="${prefix}_link">
+      <sensor type="depth" name="${prefix}">
         <always_on>true</always_on>
         <update_rate>${cam_fps}</update_rate>
@@ -53,7 +53,7 @@
           </clip>
         </camera>
-        <plugin name="camera_plugin" filename="libgazebo_ros_camera.so">
+        <plugin name="${prefix}_plugin" filename="libgazebo_ros_camera.so">
           <ros>
-            <namespace>camera</namespace>
+            <namespace>${ros_namespace}</namespace>
             <remapping>~/image_raw:=color/image_raw</remapping>
             <remapping>~/camera_info:=color/camera_info</remapping>
@@ -62,6 +62,6 @@
             <remapping>~/points:=depth/color/points</remapping>
           </ros>
-          <camera_name>camera</camera_name>
-          <frame_name>camera_color_optical_frame</frame_name>
+          <camera_name>${camera_name}</camera_name>
+          <frame_name>${prefix}_color_optical_frame</frame_name>
           <min_depth>0.1</min_depth>
           <max_depth>10.0</max_depth>

File: src/ur10e_scene/urdf/ur10e_anchored.urdf.xacro (robot description, xacro)
@@ -48,6 +48,10 @@
   </joint>
   <xacro:include filename="$(find ur10e_scene)/urdf/realsense_d435.xacro" />
-  <xacro:realsense_d435 parent="world">
+  <xacro:realsense_d435 parent="world" prefix="camera" ros_namespace="camera" camera_name="camera">
     <origin xyz="0 0 1.8" rpy="0 1.57079632679 0" />
   </xacro:realsense_d435>
+  <!-- Front overview RGB-D camera for perception experiments on the full manipulator table. -->
+  <xacro:realsense_d435 parent="world" prefix="front_camera" ros_namespace="front_camera" camera_name="camera">
+    <origin xyz="0.95 0.0 1.30" rpy="0 0.50 3.14159265359" />
+  </xacro:realsense_d435>
 </robot>
