Commit message: feat(ur10e): basic manipulation policies with URDF-based IK - URDF-based FK/Jacobian/DLS-IK (ur_kinematics.py), consistent with tf/world - UR10eInterface policies: move_to, move_to_object, pick, place, home,   forward/backward/left/right/up/down jogs, grasp/release - pull object coordinates from Gazebo (/gazebo/model_states) - kinematic grasp via /gazebo/set_entity_state (stable in Gazebo Classic) - CLI command sender; entry points; gripper controller + scene fixes - scene: correct cube/tray inertia, contact tuning, gazebo_ros_state plugin,   path-agnostic launch, optenv camera params

File: src/ur10e_scene/urdf/gripper_urdf/gripper.urdf (robot description, URDF)
Before this commit: robot linear_gripper, 3 links, 2 joints
Joints:
- joint left_jaw_joint: limit lower=0 upper=0.068 effort=120 velocity=0.05 -> lower=0 upper=0.068 effort=35 velocity=0.03
- joint right_jaw_joint: limit lower=0 upper=0.068 effort=120 velocity=0.05 -> lower=0 upper=0.068 effort=35 velocity=0.03; mimic joint=left_jaw_joint multiplier=1 offset=0 -> (none)

File: src/ur10e_scene/urdf/realsense_d435.xacro (robot description, xacro)
@@ -1,7 +1,7 @@
 <?xml version="1.0"?>
 <robot xmlns:xacro="http://ros.org/wiki/xacro">
-  <xacro:property name="cam_fps" value="$(env TARGET_VIDEO_FPS)" />
-  <xacro:property name="cam_width" value="$(env TARGET_VIDEO_WIDTH)" />
-  <xacro:property name="cam_height" value="$(env TARGET_VIDEO_HEIGHT)" />
+  <xacro:property name="cam_fps" value="$(optenv TARGET_VIDEO_FPS 30)" />
+  <xacro:property name="cam_width" value="$(optenv TARGET_VIDEO_WIDTH 640)" />
+  <xacro:property name="cam_height" value="$(optenv TARGET_VIDEO_HEIGHT 480)" />
   <xacro:macro name="realsense_d435" params="parent *origin">
     <link name="camera_link">

File: src/ur10e_scene/urdf/ur10e_anchored.urdf.xacro (robot description, xacro)
@@ -21,4 +21,25 @@
   </gazebo>
   <xacro:include filename="$(find ur10e_scene)/urdf/gripper_urdf/gripper.urdf" />
+  <ros2_control name="gripper_ros2_control" type="system">
+    <hardware>
+      <plugin>gazebo_ros2_control/GazeboSystem</plugin>
+    </hardware>
+    <joint name="left_jaw_joint">
+      <command_interface name="position">
+        <param name="min">0.0</param>
+        <param name="max">0.068</param>
+      </command_interface>
+      <state_interface name="position"/>
+      <state_interface name="velocity"/>
+    </joint>
+    <joint name="right_jaw_joint">
+      <command_interface name="position">
+        <param name="min">0.0</param>
+        <param name="max">0.068</param>
+      </command_interface>
+      <state_interface name="position"/>
+      <state_interface name="velocity"/>
+    </joint>
+  </ros2_control>
   <joint name="gripper_mount_joint" type="fixed">
     <parent link="tool0" />
